File: Hardware/KiCAD/Ingenuity.kicad_pcb (KiCad board)
At the start: 4 copper layers, 65 x 30 mm, 45 parts, among them J1 Conn_01x02, J2 Conn_02x05_Odd_Even, J3 Conn_02x20_Odd_Even, J4 Conn_01x03, J5 Conn_01x03, J6 Conn_01x02, J7 Conn_01x02, J8 Conn_ST_STDC14, Q1 NMOS, Q2 NMOS, SW1 SW_SPDT, SW2 SW_Push, U2 STM32L412KBTx, U3 AMS1117-3.3, U4 LSM6DSM

Commit message: pcb
Parts:
- removed D2, D4: LED, LED_SMD:LED_0603_1608Metric
- removed J6, J7: Conn_01x02, Connector_JST:JST_XH_B2B-XH-A_1x02_P2.50mm_Vertical
- removed Q1, Q2: NMOS, Package_TO_SOT_SMD:SOT-23
- removed R10: R_Small, Resistor_SMD:R_0402_1005Metric
- removed R3: 375, Resistor_SMD:R_0402_1005Metric
- removed R5: 250, Resistor_SMD:R_0402_1005Metric
- removed SW1: SW_SPDT, mesmodules:SW_472121010111
- added C10: 1u, Capacitor_SMD:C_0402_1005Metric, F.Cu at (174.5, 100.3)
- added C11: 100n, Capacitor_SMD:C_0402_1005Metric, F.Cu at (164.1, 120.5)
- added TP1: TestPoint, TestPoint:TestPoint_Pad_D1.5mm, F.Cu at (184.4, 105.7)
- added TP2: TestPoint, TestPoint:TestPoint_Pad_D1.5mm, F.Cu at (178.4, 104.1)
- added TP3: TestPoint, TestPoint:TestPoint_Pad_D1.5mm, F.Cu at (158.0, 113.0)
- added TP4: TestPoint, TestPoint:TestPoint_Pad_D1.5mm, F.Cu at (161.0, 113.0)
- added TP5: TestPoint, TestPoint:TestPoint_Pad_D1.5mm, F.Cu at (164.0, 113.0)
- added TP6: TestPoint, TestPoint:TestPoint_Pad_D1.5mm, F.Cu at (167.0, 113.0)
- C7: value 10u -> 100n; footprint Capacitor_SMD:C_0603_1608Metric -> Capacitor_SMD:C_0402_1005Metric
- C8: value 10u -> 1u; footprint Capacitor_SMD:C_0603_1608Metric -> Capacitor_SMD:C_0402_1005Metric
- J1: value Conn_01x02 -> Conn_01x04; footprint Connector_JST:JST_XH_B2B-XH-A_1x02_P2.50mm_Vertical -> Connector_JST:JST_XH_B4B-XH-A_1x04_P2.50mm_Vertical
- J3: moved to B.Cu
- R1: value 1k -> 27k
- R9: value R_Small -> 10k
- U1: footprint mesmodules:Buck_17395xx36 -> myemp:Buck_ing
- U3: value AMS1117-3.3 -> BU33...; footprint Package_TO_SOT_SMD:SOT-223-3_TabPin2 -> Package_TO_SOT_SMD:SOT-23-5
- moved H4 94.3 mm to (130.5, 127.5)
- moved J4 90.8 mm to (131.0, 107.5), turned to -90 degrees
- moved SW2 71.6 mm to (150.5, 109.5), turned to 90 degrees
- moved H3 68.2 mm to (190.5, 127.5)
- moved J3 62.0 mm to (184.7, 128.5)
- moved C9 58.0 mm to (166.1, 120.5), turned to 180 degrees
- moved J2 56.8 mm to (139.2, 108.4)
- moved U1 55.7 mm to (178.5, 107.8), turned to 180 degrees
- moved U4 55.6 mm to (165.1, 118.2)
- moved J5 52.3 mm to (189.5, 112.5)
- moved C3 52.0 mm to (168.5, 109.5)
- moved C1 51.2 mm to (180.2, 106.3), turned to 180 degrees
- moved R6 51.2 mm to (169.9, 96.4)
- moved D5 51.1 mm to (169.9, 93.8)
- moved C4 51.0 mm to (157.5, 104.5)
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Connections:
- C1 pad 1: +7.5V -> +6V
- C7 pad 1: +5V -> TENSION_BATTERIE
- C8 pad 1: +3.3V -> +5V
- J1 pad 1: GND -> Net-(J1-Pin_1)
- J1 pad 2: +BATT -> unconnected-(J1-Pin_2-Pad2)
- J2 pad 1: unconnected-(J2-Pin_1-Pad1) -> INT
- J2 pad 9: GND -> unconnected-(J2-Pin_9-Pad9)
- J4 pad 2: +5V -> unconnected-(J4-Pin_2-Pad2)
- J4 pad 3: PWM3 -> PWM2
- J5 pad 2: +5V -> +6V
- J5 pad 3: PWM4 -> PWM1
- R1 pad 1: Net-(SW1-A) -> TENSION_BATTERIE
- R1 pad 2: GND -> Net-(J1-Pin_1)
- R9 pad 1: PWM2 -> TENSION_BATTERIE
- R9 pad 2: Net-(Q1-G) -> GND
- U1 pad 1: +7.5V -> +6V
- U2 pad 14: unconnected-(U2-PB0-Pad14) -> TENSION_BATTERIE
- U2 pad 18: PWM4 -> unconnected-(U2-PA8-Pad18)
- U2 pad 21: PWM3 -> unconnected-(U2-PA11-Pad21)
- U2 pad 28: unconnected-(U2-PB5-Pad28) -> INT
- U3 pad 1: GND -> +5V
- U3 pad 2: +3.3V -> GND
Routing:
- net INT: track 0.00 -> 36.0 mm
- net +5V: track 2.47 -> 33.6 mm, vias 4 -> 0
- net TENSION_BATTERIE: track 0.00 -> 23.0 mm, vias 0 -> 2
- net GND: track 22.5 -> 43.9 mm, vias 39 -> 87
- net +7.5V: track 20.2 -> 0.00 mm, vias 1 -> 0
- net PWM4: track 17.8 -> 0.00 mm, vias 1 -> 0
- net +6V: track 0.00 -> 15.9 mm
- net USART1_TX: track 4.86 -> 20.0 mm, vias 0 -> 2
- net NRST: track 30.0 -> 42.5 mm, vias 3 -> 2
- net SPI_CS: track 6.76 -> 18.9 mm
- net USART1_RX: track 8.94 -> 21.0 mm, vias 0 -> 2
- net PWM3: track 11.7 -> 0.00 mm
- net PWM2: track 32.8 -> 44.1 mm
- net PWM1: track 41.1 -> 30.2 mm, vias 0 -> 1
- net USART2_RX: track 26.2 -> 35.3 mm, vias 1 -> 0
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- added copper zone on In2.Cu, net +3.3V
- added copper zone on In1.Cu, net GND
- removed copper zone on In1.Cu, net +3.3V
- removed copper zone on F.Cu, net +5V
- removed copper zone on In1.Cu, net +5V
- removed copper zone on In1.Cu, net +7.5V
- removed copper zone on B.Cu, net +BATT
- removed copper zone on B.Cu, net GND
- removed copper zone on In2.Cu, net GND
Other:
- board size 65 x 30 mm -> 68 x 40.5 mm
- board text removed: "+ Batt -"
- board text removed: "+3V3"
- board text removed: "+5V"
- board text removed: "1"
- board text removed: "Mot1"
- board text removed: "Mot2"
- board text removed: "NRST"
- board text removed: "Servo1"
- board text removed: "Servo2"
- board text removed: "Vbat"
